File: Brushograf_PCB-revB/Brushograf_PCB-revB.kicad_sch (KiCad schematic)
At the start: 81 parts, among them J1 Conn_01x05_Socket, J12 USB-C PD in, J13 FluidDial pendant, J2 Conn_01x05_Socket, J3 Conn_01x05_Socket, J5 Barrel_Jack_Switch, J6 Conn_01x07_Socket, J7 Conn_01x03_Pin, J8 SD_CARD_MICRO_AMPHENOL_114008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, Q1 AO3401A, SW1 ESP POWER, U1 ULN2003A, U2 ULN2003A, U3 ULN2003A, U4 ESP32-DevKitC, U6 CH224K, U7 TPS54202, U8 TPS54202

Commit message: USB-C as the only inlet; lever switch and RJ-12 placed on the board edges
Grows the outline 25mm along the top (198x48 -> 198x73mm) and places every
new part. The RJ-12 needs ~19mm behind the top edge and the old board had
11mm before the back-side SPI tracks, which is what forced the growth.
Everything from rev A keeps its coordinates.

  - The barrel jack is now gone, with its reverse-polarity FET, zener and
    gate resistor. USB-C is the sole power inlet: VBUS through a 1.5A
    polyfuse straight to the rail feeding both converters.
  - J12 sits on the left edge, receptacle overhanging it.
  - SW1 becomes an NKK GW12L panel lever switch on the left edge with the
    actuator overhanging, replacing the DIP slide. It is a 1P2T used as a
    break: common to the ESP32, one throw to the board 5V, the other open.
  - J13 RJ-12 sits on the upper edge, opening facing off the board.

Copper pours are grown with the outline and refilled, so the new strip is
poured rather than stopping partway up it.

Placement was validated against a 0.25mm occupancy model of the existing
copper, and every non-J12 DRC error is inherited unchanged from rev A.

J12 reports 27 shorting_items and 4 hole_clearance errors that are NOT
caused by the placement: the same 31 appear with the untouched stock
footprint alone on an empty board. The pads have real 0.2-0.7mm gaps and
nothing bridges them; zones, solder mask and neighbouring copper were each
ruled out by experiment, and every USB-C footprint in the KiCad library has
sub-0.25mm pad gaps. Flagged in the README to look at in the GUI.

53 ratsnest connections remain to be routed.

Co-Authored-By: Claude Opus 5 <noreply@anthropic.com>
Parts:
- removed D13: BZX84C10, Diode_SMD:D_SOD-123, symbol Device:D_Zener
- removed D15, D16: SS34, Diode_SMD:D_SMA_Handsoldering, symbol Device:D_Schottky
- removed J5: Barrel_Jack_Switch, Connector_BarrelJack:BarrelJack_Horizontal, symbol Connector:Barrel_Jack_Switch
- removed Q1: AO3401A, Package_TO_SOT_SMD:SOT-23, symbol Transistor_FET:AO3401A
- removed R21: 100k, Resistor_SMD:R_1206_3216Metric_Pad1.30x1.75mm_HandSolder, symbol Device:R
- removed SW1: ESP POWER, Button_Switch_THT:SW_DIP_SPSTx01_Slide_9.78x4.72mm_W7.62mm_P2.54mm, symbol Switch:SW_SPST
- added SW1: ESP POWER, Button_Switch_THT:SW_Lever_1P2T_NKK_GW12LxH, symbol Switch:SW_SPDT
- C7: value 10uF/50V -> 10uF/35V
Connections:
- net VIN is gone; now on net VBUS: F1.1
- net VIN_DC is gone; now on net VSUP: C7.1
- net 5V_SYS: now also SW1.2 (B)
- net VSUP: now also F1.2
- net at D14.1 (K): now also SW1.1 (A)
- no-connect marks 6 -> 7
Other:
- moved on the sheet: C10
